Commit message: 先引入slam_toolbox建图验证规划算法,保存room.world文件

File: src/mbot_pkg/urdf/mbot_base.urdf.xacro (robot description, xacro)
@@ -1,4 +1,4 @@
 <?xml version="1.0"?>
-<robot name="mbot" xmlns:xacro="http://www.ros.org/wiki/xacro">
+<xacro:macro name="mbot_base" xmlns:xacro="http://www.ros.org/wiki/xacro">
   <!-- 常量定义 -->
   <xacro:property name="wheel_radius" value="0.05" />
@@ -197,3 +197,3 @@
     <origin xyz="0 0 0" rpy="0 0 0" />
   </joint>
-</robot>
+</xacro:macro>

File: src/mbot_pkg/urdf/mbot_gazebo.urdf.xacro (robot description, xacro)
@@ -3,4 +3,5 @@
   <!-- 包含基础结构 -->
   <xacro:include filename="mbot_base.urdf.xacro" />
+  <!-- <xacro:mbot_base /> -->
   <!-- Gazebo插件配置 -->
   <gazebo>
@@ -20,4 +21,16 @@
       <publish_odom_tf>true</publish_odom_tf>
       <publish_wheel_tf>true</publish_wheel_tf>
+    </plugin>
+  </gazebo>
+  <gazebo>
+    <plugin name="ground_truth_plugin" filename="libgazebo_ros_p3d.so">
+       <ros>
+            <namespace>/mbot</namespace>
+            <remapping>odom:=gazebo_pose</remapping>
+       </ros>
+      <frame_name>world</frame_name>
+      <body_name>base_link</body_name>
+      <update_rate>50.0</update_rate>
+      <gaussian_noise>0</gaussian_noise>
     </plugin>
   </gazebo>

Commit message: PID控制TBD slam发布预定地图和位姿 navigation发布固定轨迹 pid循迹暂时未完成

File: src/mbot_pkg/urdf/mbot_base.urdf.xacro (robot description, xacro)
@@ -19,4 +19,12 @@
     <color rgba="0.0 0.0 0.0 1.0" />
   </material>
+  <!-- 新增：base_footprint（地面投影坐标系，z=0） -->
+  <link name="base_footprint">
+    <!-- 虚拟坐标系，无需视觉/碰撞模型 -->
+    <inertial>
+      <mass value="0.001" /> <!-- 极小质量，避免动力学问题 -->
+      <inertia ixx="1e-6" ixy="0" ixz="0" iyy="1e-6" iyz="0" izz="1e-6" />
+    </inertial>
+  </link>
   <!-- 底盘 -->
   <link name="base_link">
@@ -148,4 +156,12 @@
     </inertial>
   </link>
+   <!-- 新增：base_footprint到base_link的固定关节 -->
+  <joint name="base_footprint_joint" type="fixed">
+    <parent link="base_footprint" /> <!-- 父级：地面坐标系 -->
+    <child link="base_link" />       <!-- 子级：机器人本体 -->
+    <!-- z方向偏移：确保base_footprint在地面（z=0），base_link在其上方 -->
+    <!-- 计算方式：轮子半径（0.05） + 底盘高度的一半（0.05/2） -->
+    <origin xyz="0 0 ${wheel_radius + base_height/2}" rpy="0 0 0" />
+  </joint>
   <!-- 左轮关节 -->
   <joint name="left_wheel_joint" type="continuous">
@@ -194,5 +210,5 @@
   <joint name="odom_joint" type="fixed">
     <parent link="odom" />
-    <child link="base_link" />
+    <child link="base_footprint" />
     <origin xyz="0 0 0" rpy="0 0 0" />
   </joint>

File: src/mbot_pkg/urdf/mbot_gazebo.urdf.xacro (robot description, xacro)
@@ -12,4 +12,5 @@
         <remapping>odom:=odom</remapping>
       </ros>
+      <base_link>base_footprint</base_link>
       <wheel_separation>${wheel_separation}</wheel_separation>
       <wheel_diameter>${wheel_radius * 2}</wheel_diameter>
@@ -21,16 +22,4 @@
       <publish_odom_tf>true</publish_odom_tf>
       <publish_wheel_tf>true</publish_wheel_tf>
-    </plugin>
-  </gazebo>
-  <gazebo>
-    <plugin name="ground_truth_plugin" filename="libgazebo_ros_p3d.so">
-       <ros>
-            <namespace>/mbot</namespace>
-            <remapping>odom:=gazebo_pose</remapping>
-       </ros>
-      <frame_name>world</frame_name>
-      <body_name>base_link</body_name>
-      <update_rate>50.0</update_rate>
-      <gaussian_noise>0</gaussian_noise>
     </plugin>
   </gazebo>

Commit message: PID微调,增加积分限幅与积分分离

File: src/mbot_pkg/urdf/mbot_base.urdf.xacro (robot description, xacro)
@@ -120,5 +120,5 @@
     <collision>
       <geometry>
-        <cylinder radius="${lidar_radius}" length="${lidar_radius}" />
+        <cylinder radius="${lidar_radius}" length="${lidar_height}" />
       </geometry>
       <origin xyz="0 0 0" rpy="0 0 0" />
